File: pcb/pcb.kicad_pcb (KiCad board)
At the start: 2 copper layers, 285 x 95.1 mm, 142 parts, among them SW1 SW_Push, U1 PRTR5V0U2X, U2 ATmega32U4-AU, Y1 16MHz

Commit message: pcb WIP
Parts:
- C1, C2, C3, C4, C5, C6, C7, D10, D11, D16, D20, D21, D22, D23, D24, D25, D27, D28, D29, D30, D33, D34, D51, D7, D8, F1, R1, R2, R3, R4, R5, R6, SW1, U1, U2, Y1: moved to B.Cu
- moved F1 440.6 mm to (38.7, 144.6), turned to 180 degrees
- moved R6 437.4 mm to (40.3, 147.7), turned to 180 degrees
- moved D7 436.8 mm to (53.2, 59.5), turned to 90 degrees
- moved D10 405.0 mm to (79.4, 33.3), turned to 90 degrees
- moved D11 392.1 mm to (88.9, 52.4), turned to 90 degrees
- moved D8 383.4 mm to (74.6, 71.4), turned to 90 degrees
- moved D16 381.6 mm to (108.0, 52.4), turned to 90 degrees
- moved C4 380.2 mm to (69.1, 173.7), turned to 180 degrees
- moved C1 377.7 mm to (70.4, 177.1), turned to 180 degrees
- moved C2 368.8 mm to (74.8, 180.1), turned to 180 degrees
- moved C3 368.8 mm to (74.8, 177.1), turned to 180 degrees
- moved D20 367.7 mm to (127.0, 52.4), turned to 90 degrees
- moved D23 362.8 mm to (136.5, 33.3), turned to 90 degrees
- moved D21 356.8 mm to (131.8, 71.4), turned to 90 degrees
- moved D22 356.8 mm to (122.2, 90.5), turned to 90 degrees
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Connections:
- MX1 pad 2: Net-(D1-Pad2) -> Net-(MX1-Pad2)
- MX10 pad 2: Net-(D10-Pad2) -> Net-(MX10-Pad2)
- MX11 pad 2: Net-(D11-Pad2) -> Net-(MX11-Pad2)
- MX12 pad 2: Net-(D12-Pad2) -> Net-(MX12-Pad2)
- MX13 pad 2: Net-(D13-Pad2) -> Net-(MX13-Pad2)
- MX14 pad 2: Net-(D14-Pad2) -> Net-(MX14-Pad2)
- MX15 pad 2: Net-(D15-Pad2) -> Net-(MX15-Pad2)
- MX16 pad 2: Net-(D16-Pad2) -> Net-(MX16-Pad2)
- MX17 pad 2: Net-(D17-Pad2) -> Net-(MX17-Pad2)
- MX18 pad 2: Net-(D18-Pad2) -> Net-(MX18-Pad2)
- MX19 pad 2: Net-(D19-Pad2) -> Net-(MX19-Pad2)
- MX2 pad 2: Net-(D2-Pad2) -> Net-(MX2-Pad2)
- MX20 pad 2: Net-(D20-Pad2) -> Net-(MX20-Pad2)
- MX21 pad 2: Net-(D21-Pad2) -> Net-(MX21-Pad2)
- MX22 pad 2: Net-(D22-Pad2) -> Net-(MX22-Pad2)
- MX23 pad 2: Net-(D23-Pad2) -> Net-(MX23-Pad2)
- MX24 pad 2: Net-(D24-Pad2) -> Net-(MX24-Pad2)
- MX25 pad 2: Net-(D25-Pad2) -> Net-(MX25-Pad2)
- MX26 pad 2: Net-(D26-Pad2) -> Net-(MX26-Pad2)
- MX27 pad 2: Net-(D27-Pad2) -> Net-(MX27-Pad2)
- MX28 pad 2: Net-(D28-Pad2) -> Net-(MX28-Pad2)
- MX29 pad 2: Net-(D29-Pad2) -> Net-(MX29-Pad2)
- MX3 pad 2: Net-(D3-Pad2) -> Net-(MX3-Pad2)
- MX30 pad 2: Net-(D30-Pad2) -> Net-(MX30-Pad2)
- MX31 pad 2: Net-(D31-Pad2) -> Net-(MX31-Pad2)
- MX32 pad 2: Net-(D32-Pad2) -> Net-(MX32-Pad2)
- MX33 pad 2: Net-(D33-Pad2) -> Net-(MX33-Pad2)
- MX34 pad 2: Net-(D34-Pad2) -> Net-(MX34-Pad2)
- MX35 pad 2: Net-(D35-Pad2) -> Net-(MX35-Pad2)
- MX36 pad 2: Net-(D36-Pad2) -> Net-(MX36-Pad2)
- MX37 pad 2: Net-(D37-Pad2) -> Net-(MX37-Pad2)
- MX38 pad 2: Net-(D38-Pad2) -> Net-(MX38-Pad2)
- MX39 pad 2: Net-(D39-Pad2) -> Net-(MX39-Pad2)
- MX4 pad 2: Net-(D4-Pad2) -> Net-(MX4-Pad2)
- MX40 pad 2: Net-(D40-Pad2) -> Net-(MX40-Pad2)
- MX41 pad 2: Net-(D41-Pad2) -> Net-(MX41-Pad2)
- MX42 pad 2: Net-(D42-Pad2) -> Net-(MX42-Pad2)
- MX43 pad 2: Net-(D43-Pad2) -> Net-(MX43-Pad2)
- MX44 pad 2: Net-(D44-Pad2) -> Net-(MX44-Pad2)
- MX45 pad 2: Net-(D45-Pad2) -> Net-(MX45-Pad2)
- MX46 pad 2: Net-(D46-Pad2) -> Net-(MX46-Pad2)
- MX47 pad 2: Net-(D47-Pad2) -> Net-(MX47-Pad2)
- MX48 pad 2: Net-(D48-Pad2) -> Net-(MX48-Pad2)
- MX49 pad 2: Net-(D49-Pad2) -> Net-(MX49-Pad2)
- MX5 pad 2: Net-(D5-Pad2) -> Net-(MX5-Pad2)
- MX50 pad 2: Net-(D50-Pad2) -> Net-(MX50-Pad2)
- MX51 pad 2: Net-(D51-Pad2) -> Net-(MX51-Pad2)
- MX52 pad 2: Net-(D52-Pad2) -> Net-(MX52-Pad2)
- MX53 pad 2: Net-(D53-Pad2) -> Net-(MX53-Pad2)
- MX54 pad 2: Net-(D54-Pad2) -> Net-(MX54-Pad2)
- MX55 pad 2: Net-(D55-Pad2) -> Net-(MX55-Pad2)
- MX56 pad 2: Net-(D56-Pad2) -> Net-(MX56-Pad2)
- MX57 pad 2: Net-(D57-Pad2) -> Net-(MX57-Pad2)
- MX58 pad 2: Net-(D58-Pad2) -> Net-(MX58-Pad2)
- MX59 pad 2: Net-(D59-Pad2) -> Net-(MX59-Pad2)
- MX6 pad 2: Net-(D6-Pad2) -> Net-(MX6-Pad2)
- MX60 pad 2: Net-(D60-Pad2) -> Net-(MX60-Pad2)
- MX61 pad 2: Net-(D61-Pad2) -> Net-(MX61-Pad2)
- MX7 pad 2: Net-(D7-Pad2) -> Net-(MX7-Pad2)
- MX8 pad 2: Net-(D8-Pad2) -> Net-(MX8-Pad2)
- MX9 pad 2: Net-(D9-Pad2) -> Net-(MX9-Pad2)
- U1 pad 1: GND -> Net-(U1-Pad1)
- U1 pad 2: Net-(R4-Pad2) -> Net-(U1-Pad2)
- U1 pad 3: Net-(R3-Pad2) -> Net-(U1-Pad3)
- U1 pad 4: VCC -> Net-(U1-Pad4)
- USB1 pad 1: GND -> Net-(USB1-Pad1)
- USB1 pad 10: Net-(R2-Pad2) -> Net-(USB1-Pad10)
- USB1 pad 11: VCC -> Net-(USB1-Pad11)
- USB1 pad 12: GND -> Net-(USB1-Pad1)
- USB1 pad 13: GND -> Net-(USB1-Pad1)
- USB1 pad 2: VCC -> Net-(USB1-Pad11)
- USB1 pad 4: Net-(R1-Pad2) -> Net-(USB1-Pad4)
- USB1 pad 5: Net-(R3-Pad2) -> Net-(U1-Pad3)
- USB1 pad 6: Net-(R4-Pad2) -> Net-(U1-Pad2)
- USB1 pad 7: Net-(R3-Pad2) -> Net-(U1-Pad3)
- USB1 pad 8: Net-(R4-Pad2) -> Net-(U1-Pad2)
Routing:
- net Net-(USB1-Pad1): track 0.00 -> 19.9 mm
- net Net-(U1-Pad3): track 0.00 -> 3.00 mm
- net Net-(U1-Pad2): track 0.00 -> 2.99 mm
- added copper zone on B.Cu, net (none)
Other:
- net class Power added: clearance 0.2, trace_width 0.381, via_dia 0.8, via_drill 0.4

Commit message: PCB WIP
Parts:
- moved U1 223.6 mm to (43.2, 32.8), turned to 270 degrees
- moved R1 220.2 mm to (36.3, 31.0), turned to 270 degrees
- moved R4 218.6 mm to (43.8, 39.2), turned to 90 degrees
- moved R2 218.0 mm to (48.1, 31.2)
- moved R3 208.6 mm to (41.8, 39.2), turned to 90 degrees
- moved R5 142.2 mm to (117.9, 99.9)
- moved F1 106.6 mm to (34.0, 38.1), turned to 90 degrees
- moved C6 97.6 mm to (129.4, 104.4), turned to 90 degrees
- moved C1 96.2 mm to (123.7, 97.0), turned to 90 degrees
- moved R6 95.0 mm to (129.2, 114.0), turned to 90 degrees
- moved C2 93.5 mm to (117.5, 96.9), turned to 270 degrees
- moved C5 93.0 mm to (111.4, 108.7), turned to 270 degrees
- moved C7 89.7 mm to (109.3, 108.7), turned to 270 degrees
- moved C3 79.2 mm to (125.7, 116.5)
- moved C4 74.6 mm to (117.1, 116.6), turned to 0 degrees
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Connections:
- MX1 pad 2: Net-(MX1-Pad2) -> Net-(D1-Pad2)
- MX10 pad 2: Net-(MX10-Pad2) -> Net-(D10-Pad2)
- MX11 pad 2: Net-(MX11-Pad2) -> Net-(D11-Pad2)
- MX12 pad 2: Net-(MX12-Pad2) -> Net-(D12-Pad2)
- MX13 pad 2: Net-(MX13-Pad2) -> Net-(D13-Pad2)
- MX14 pad 2: Net-(MX14-Pad2) -> Net-(D14-Pad2)
- MX15 pad 2: Net-(MX15-Pad2) -> Net-(D15-Pad2)
- MX16 pad 2: Net-(MX16-Pad2) -> Net-(D16-Pad2)
- MX17 pad 2: Net-(MX17-Pad2) -> Net-(D17-Pad2)
- MX18 pad 2: Net-(MX18-Pad2) -> Net-(D18-Pad2)
- MX19 pad 2: Net-(MX19-Pad2) -> Net-(D19-Pad2)
- MX2 pad 2: Net-(MX2-Pad2) -> Net-(D2-Pad2)
- MX20 pad 2: Net-(MX20-Pad2) -> Net-(D20-Pad2)
- MX21 pad 2: Net-(MX21-Pad2) -> Net-(D21-Pad2)
- MX22 pad 2: Net-(MX22-Pad2) -> Net-(D22-Pad2)
- MX23 pad 2: Net-(MX23-Pad2) -> Net-(D23-Pad2)
- MX24 pad 2: Net-(MX24-Pad2) -> Net-(D24-Pad2)
- MX25 pad 2: Net-(MX25-Pad2) -> Net-(D25-Pad2)
- MX26 pad 2: Net-(MX26-Pad2) -> Net-(D26-Pad2)
- MX27 pad 2: Net-(MX27-Pad2) -> Net-(D27-Pad2)
- MX28 pad 2: Net-(MX28-Pad2) -> Net-(D28-Pad2)
- MX29 pad 2: Net-(MX29-Pad2) -> Net-(D29-Pad2)
- MX3 pad 2: Net-(MX3-Pad2) -> Net-(D3-Pad2)
- MX30 pad 2: Net-(MX30-Pad2) -> Net-(D30-Pad2)
- MX31 pad 2: Net-(MX31-Pad2) -> Net-(D31-Pad2)
- MX32 pad 2: Net-(MX32-Pad2) -> Net-(D32-Pad2)
- MX33 pad 2: Net-(MX33-Pad2) -> Net-(D33-Pad2)
- MX34 pad 2: Net-(MX34-Pad2) -> Net-(D34-Pad2)
- MX35 pad 2: Net-(MX35-Pad2) -> Net-(D35-Pad2)
- MX36 pad 2: Net-(MX36-Pad2) -> Net-(D36-Pad2)
- MX37 pad 2: Net-(MX37-Pad2) -> Net-(D37-Pad2)
- MX38 pad 2: Net-(MX38-Pad2) -> Net-(D38-Pad2)
- MX39 pad 2: Net-(MX39-Pad2) -> Net-(D39-Pad2)
- MX4 pad 2: Net-(MX4-Pad2) -> Net-(D4-Pad2)
- MX40 pad 2: Net-(MX40-Pad2) -> Net-(D40-Pad2)
- MX41 pad 2: Net-(MX41-Pad2) -> Net-(D41-Pad2)
- MX42 pad 2: Net-(MX42-Pad2) -> Net-(D42-Pad2)
- MX43 pad 2: Net-(MX43-Pad2) -> Net-(D43-Pad2)
- MX44 pad 2: Net-(MX44-Pad2) -> Net-(D44-Pad2)
- MX45 pad 2: Net-(MX45-Pad2) -> Net-(D45-Pad2)
- MX46 pad 2: Net-(MX46-Pad2) -> Net-(D46-Pad2)
- MX47 pad 2: Net-(MX47-Pad2) -> Net-(D47-Pad2)
- MX48 pad 2: Net-(MX48-Pad2) -> Net-(D48-Pad2)
- MX49 pad 2: Net-(MX49-Pad2) -> Net-(D49-Pad2)
- MX5 pad 2: Net-(MX5-Pad2) -> Net-(D5-Pad2)
- MX50 pad 2: Net-(MX50-Pad2) -> Net-(D50-Pad2)
- MX51 pad 2: Net-(MX51-Pad2) -> Net-(D51-Pad2)
- MX52 pad 2: Net-(MX52-Pad2) -> Net-(D52-Pad2)
- MX53 pad 2: Net-(MX53-Pad2) -> Net-(D53-Pad2)
- MX54 pad 2: Net-(MX54-Pad2) -> Net-(D54-Pad2)
- MX55 pad 2: Net-(MX55-Pad2) -> Net-(D55-Pad2)
- MX56 pad 2: Net-(MX56-Pad2) -> Net-(D56-Pad2)
- MX57 pad 2: Net-(MX57-Pad2) -> Net-(D57-Pad2)
- MX58 pad 2: Net-(MX58-Pad2) -> Net-(D58-Pad2)
- MX59 pad 2: Net-(MX59-Pad2) -> Net-(D59-Pad2)
- MX6 pad 2: Net-(MX6-Pad2) -> Net-(D6-Pad2)
- MX60 pad 2: Net-(MX60-Pad2) -> Net-(D60-Pad2)
- MX61 pad 2: Net-(MX61-Pad2) -> Net-(D61-Pad2)
- MX7 pad 2: Net-(MX7-Pad2) -> Net-(D7-Pad2)
- MX8 pad 2: Net-(MX8-Pad2) -> Net-(D8-Pad2)
- MX9 pad 2: Net-(MX9-Pad2) -> Net-(D9-Pad2)
- U1 pad 1: Net-(U1-Pad1) -> GND
- U1 pad 2: Net-(U1-Pad2) -> Net-(R4-Pad2)
- U1 pad 3: Net-(U1-Pad3) -> Net-(R3-Pad2)
- U1 pad 4: Net-(U1-Pad4) -> VCC
- USB1 pad 1: Net-(USB1-Pad1) -> GND
- USB1 pad 10: Net-(USB1-Pad10) -> Net-(R2-Pad2)
- USB1 pad 11: Net-(USB1-Pad11) -> VCC
- USB1 pad 12: Net-(USB1-Pad1) -> GND
- USB1 pad 13: Net-(USB1-Pad1) -> GND
- USB1 pad 2: Net-(USB1-Pad11) -> VCC
- USB1 pad 4: Net-(USB1-Pad4) -> Net-(R1-Pad2)
- USB1 pad 5: Net-(U1-Pad3) -> Net-(R3-Pad2)
- USB1 pad 6: Net-(U1-Pad2) -> Net-(R4-Pad2)
- USB1 pad 7: Net-(U1-Pad3) -> Net-(R3-Pad2)
- USB1 pad 8: Net-(U1-Pad2) -> Net-(R4-Pad2)
Routing:
- net GND: track 0.00 -> 102.1 mm
- net +5V: track 0.00 -> 51.4 mm, vias 0 -> 3
- net VCC: track 0.00 -> 21.5 mm, vias 0 -> 3
- net Net-(USB1-Pad1): track 19.9 -> 0.00 mm
- net Net-(R4-Pad2): track 0.00 -> 12.0 mm
- net Net-(R3-Pad2): track 0.00 -> 10.8 mm
- net Net-(C2-Pad1): track 0.00 -> 10.2 mm
- net Net-(R5-Pad2): track 0.00 -> 8.35 mm
- net Net-(C1-Pad1): track 0.34 -> 7.38 mm
- net Net-(C7-Pad1): track 0.00 -> 6.80 mm
- net Net-(R1-Pad2): track 0.00 -> 6.63 mm
- net Net-(R2-Pad2): track 0.00 -> 4.17 mm
- net Net-(U1-Pad3): track 3.00 -> 0.00 mm
- net Net-(U1-Pad2): track 2.99 -> 0.00 mm
- net Net-(R6-Pad2): track 0.00 -> 2.18 mm

Commit message: PCB WIP
Parts:
- moved SW1 17.4 mm to (128.2, 96.6), turned to 0 degrees
- moved R6 17.0 mm to (112.2, 114.9), turned to 0 degrees
- moved C3 16.7 mm to (109.8, 111.4), turned to 90 degrees
- moved C7 15.9 mm to (117.5, 95.1), turned to 180 degrees
- moved C4 15.7 mm to (109.6, 102.8), turned to 270 degrees
- moved C1 13.6 mm to (129.3, 109.4), turned to 0 degrees
- moved C2 13.4 mm to (129.3, 103.2), turned to 180 degrees
- moved C6 13.1 mm to (121.8, 115.1), turned to 0 degrees
- moved C5 13.1 mm to (117.5, 97.1), turned to 180 degrees
- moved Y1 12.7 mm to (129.3, 106.3), turned to 90 degrees
- moved R5 9.16 mm to (126.3, 103.6), turned to 90 degrees
- moved U2 4.27 mm to (117.5, 107.2), turned to 270 degrees
Routing:
- net row0: track 0.00 -> 282.1 mm
- net row4: track 0.00 -> 274.3 mm
- net row2: track 0.00 -> 258.6 mm
- net row1: track 0.00 -> 254.7 mm
- net row3: track 0.00 -> 245.0 mm
- net D+: track 0.00 -> 143.2 mm, vias 0 -> 4
- net D-: track 0.00 -> 138.7 mm, vias 0 -> 4
- net +5V: track 51.4 -> 175.1 mm, vias 3 -> 5
- net col13: track 0.00 -> 114.2 mm, vias 0 -> 6
- net col10: track 0.00 -> 96.2 mm, vias 0 -> 5
- net col2: track 0.00 -> 90.4 mm, vias 0 -> 5
- net col6: track 0.00 -> 87.4 mm, vias 0 -> 5
- net col11: track 0.00 -> 87.2 mm, vias 0 -> 5
- net col1: track 0.00 -> 83.3 mm, vias 0 -> 6
- net col0: track 0.00 -> 81.9 mm, vias 0 -> 2
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
Commit message: wip
Routing:
- net GND: track 104.5 -> 245.8 mm, vias 2 -> 7
- net col9: track 67.0 -> 162.4 mm, vias 4 -> 7
- net col0: track 81.9 -> 175.9 mm, vias 2 -> 6
- net col7: track 67.0 -> 129.4 mm, vias 4 -> 5
- net col1: track 83.3 -> 142.7 mm, vias 6 -> 7
- net col2: track 90.4 -> 127.4 mm
- net col3: track 67.2 -> 104.0 mm, vias 4 -> 5
- net col6: track 87.4 -> 113.9 mm
- net col4: track 67.4 -> 89.2 mm, vias 4 -> 5
- net col5: track 67.1 -> 88.4 mm, vias 4 -> 5
- net row4: track 274.3 -> 277.9 mm

Commit message: finished rev 1 PCB
Connections:
- U2 pad 1: Net-(U2-Pad1) -> row0
- U2 pad 10: Net-(U2-Pad10) -> row1
- U2 pad 11: Net-(U2-Pad11) -> row3
- U2 pad 18: Net-(U2-Pad18) -> col6
- U2 pad 19: Net-(U2-Pad19) -> col5
- U2 pad 20: Net-(U2-Pad20) -> col7
- U2 pad 21: Net-(U2-Pad21) -> col9
- U2 pad 22: Net-(U2-Pad22) -> col8
- U2 pad 25: Net-(U2-Pad25) -> col10
- U2 pad 26: Net-(U2-Pad26) -> col11
- U2 pad 27: Net-(U2-Pad27) -> col12
- U2 pad 28: Net-(U2-Pad28) -> col13
- U2 pad 31: Net-(U2-Pad31) -> col0
- U2 pad 32: Net-(U2-Pad32) -> row4
- U2 pad 36: Net-(U2-Pad36) -> col2
- U2 pad 38: Net-(U2-Pad38) -> col1
- U2 pad 39: Net-(U2-Pad39) -> row2
- U2 pad 40: Net-(U2-Pad40) -> col4
- U2 pad 41: Net-(U2-Pad41) -> col3
Routing:
- net col13: track 114.2 -> 294.9 mm, vias 6 -> 7
- net col12: track 81.1 -> 245.7 mm, vias 3 -> 4
- net col11: track 87.2 -> 219.5 mm, vias 5 -> 11
- net col10: track 96.2 -> 216.4 mm, vias 5 -> 9
- net col8: track 67.2 -> 140.5 mm, vias 4 -> 7
- net row0: track 282.1 -> 352.4 mm, vias 0 -> 4
- net row1: track 254.7 -> 305.6 mm, vias 0 -> 2
- net row2: track 258.6 -> 293.6 mm, vias 0 -> 2
- net row3: track 245.0 -> 254.9 mm, vias 0 -> 2
- net col1: track 142.7 -> 146.6 mm, vias 7 -> 9
- net col5: track 88.4 -> 90.1 mm
- net col9: track 162.4 -> 163.8 mm
- net col7: track 129.4 -> 130.7 mm
- net col2: track 127.4 -> 128.5 mm
- net col4: track 89.2 -> 90.4 mm
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Other:
- board text added: "Huskey60 rev1.0 by Huskeyboards"
